File: Eagle/V2.1/PowerMeterCurrent.sch (EAGLE design)
At the start: 59 parts, among them IC1 4067D, IC2 4514D, X1 STEREOJACK, X10 STEREOJACK, X11 STEREOJACK, X12 STEREOJACK, X13 STEREOJACK, X14 STEREOJACK, X15 STEREOJACK, X16 STEREOJACK, X2 STEREOJACK, X3 STEREOJACK, X4 STEREOJACK, X5 STEREOJACK, X6 STEREOJACK, X7 STEREOJACK, X8 STEREOJACK, X9 STEREOJACK

Commit message: Fixed BOM for current board
Parts:
- IC2: PARTNO 74HC154D,652 -> 74HC4514D,652
Changed lines of the file:
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@@
 <part name="GND" library="supply2" deviceset="GND" device=""/>
 <part name="IC2" library="45xx" deviceset="4514" device="D">
-<attribute name="PARTNO" value="74HC154D,652"/>
+<attribute name="PARTNO" value="74HC4514D,652"/>
 </part>
 <part name="LED1" library="eagle-ltspice" deviceset="LED_E" device="" value="green">
