File: Eagle/V2.2/PowerMeter.sch (EAGLE design)
At the start: 52 parts, among them IC1 4052D, IC2 74HC138D, IC3 LMV321M5, Q1 4.096MHz, X2 RASPI_BOARD_B+_E4

Commit message: Added V2.2 Eagle files and removed old versions due to hardware bug
Parts:
- removed C15: 1uF, rcl:C-EUC1206
- removed F5: MF-RM055/240-2, fuse:FUSETE5
- removed JP2: (no value), SparkFun-Connectors:M04SCREW
- removed PWR: green, eagle-ltspice:LED_E
- removed U$2, U$3: TV16E, CraigJensen:TV16E
- removed U$4: VSK-S10, CraigJensen:VSK-S10
- removed U$5: CS5463, Cirrus_Logic_By_element14_Batch_1:CS5463
- removed X2: RASPI_BOARD_B+_E4, raspberrypi_bastelstube_v13:RASPI_BOARD_B+_E4
- added F2, F3: MF-RM055/240-2, fuse:FUSETE5
- added LED1: green, eagle-ltspice:LED_E
- added PS1: VSK-S10, CraigJensen:VSK-S10
- added R17, R18: 59k, resistor:R-US_R1206
- added R19, R20: 1k, resistor:R-US_R1206
- added R21: 10K, resistor:R-US_R1206
- added T1, T2, T3: TV16E, CraigJensen:TV16E
- added X1: RASPI_BOARD_B+_E4, raspberrypi_bastelstube_v13:RASPI_BOARD_B+_E4
- C1: PARTNO (none) -> C1206C104K5RAC7867
- C10, C4: value 220pF -> .1uF; PARTNO (none) -> C1206C104K5RAC7867
- C11: value .1 uF -> 220pF; PARTNO (none) -> C1206C221J5GACTU
- C12, C8: value .1uF -> 220pF; PARTNO (none) -> C1206C221J5GACTU
- C13: PARTNO (none) -> C1206C223K5RACTU
- C14: value 22nF -> .1uF; PARTNO (none) -> C1206C104K5RAC7867
- C2: value 10u -> .1uF; device Discrete:CAP-AVX-C -> rcl:C-EUC1206; PARTNO (none) -> C1206C104K5RAC7867
- C3: value 220pF -> 10u; device rcl:C-EUC1206 -> Discrete:CAP-AVX-C; PARTNO (none) -> T491C106K016AT
- C5: value .1 uF -> 220uF; device rcl:C-EUC1206 -> adafruit:CPOL-USE2,5-6E; PARTNO (none) -> ESH227M016AE3AA
- C6: value .1 uF -> .1uF; PARTNO (none) -> C1206C104K5RAC7867
- C7: value 220uF -> 220pF; device adafruit:CPOL-USE2,5-6E -> rcl:C-EUC1206; PARTNO (none) -> C1206C221J5GACTU
- C9: value 220pF -> 22nF; PARTNO (none) -> C1206C223K5RACTU
- D1: PARTNO (none) -> P6KE6.8A
- F1: PARTNO (none) -> 0ZCC0110AF2C
- F4: PARTNO (none) -> MF-RM055/240-2
- H1, H2, H3, H4: BOM (none) -> EXCLUDE
- IC1: value 4052D -> 74HC138D; device 40xx:4052D -> 74xx-eu:74HC138D; PARTNO (none) -> SN74HC138NSR
- IC2: value 74HC138D -> 4052D; device 74xx-eu:74HC138D -> 40xx:4052D; PARTNO (none) -> CD4052BNSR
- IC3: value LMV321M5 -> CS5463; device linear:LMV321M5 -> Cirrus_Logic_By_element14_Batch_1:CS5463; PARTNO (none) -> CS5463-ISZ
- JP1: value (none) -> ACIN; device jumper:JP2E -> SparkFun-Connectors:M05; PARTNO (none) -> 1935190
- Q1: PARTNO (none) -> 9B-4.096MBBK-B
- R1, R2: value 1k -> 158; PARTNO (none) -> RC1206FR-07158RL
- R10, R11, R12, R13, R6, R8, R9: PARTNO (none) -> RC1206FR-071KL
- R14, R15: value 10K -> 59k; PARTNO (none) -> RC1206FR-071KL
- R16: value 56K -> 59k; PARTNO (none) -> RC1206FR-071KL
- R3: value 120 -> 158; PARTNO (none) -> RC1206FR-07158RL
- R4: value 120 -> 270; PARTNO (none) -> RC1206FR-07270RL
- R5: value 270 -> 1k; PARTNO (none) -> RC1206FR-071KL
- R7: value 1k -> 59k; PARTNO (none) -> RC1206FR-071KL
- SV1: value (none) -> Current Brd Connector; PARTNO (none) -> PPTC082LFBN-RC
Connections:
- removed net AC-A: F4.1, R12.1, U$4.AC(L)
- removed net AC-B: F5.1, R13.1, U$4.AC(N)
- removed net AC1: R8.2, U$3.1
- removed net BIAS: IC1A.X0, IC1A.X1, JP1.2, R3.1, R4.1, R6.1, SV1.15, U$2.3, U$3.3
- removed net IIN: R7.1, SV1.16
- removed net N: JP2.3, U$2.2, U$3.2
- removed net N$43: R10.1, R12.2
- removed net N$44: R10.2, R8.1
- removed net N$48: R11.1, R13.2
- removed net N$49: R11.2, R9.1
- removed net N$51: R9.2, U$2.1
- removed net VIN-A: IC1A.Y1, IC1A.Y2, R3.2, U$2.4
- removed net VIN-B: IC1A.X2, IC1A.Y0, R4.2, U$3.4
- new net AC(L): F2.1, PS1.AC(L), R18.1
- new net AC(N): JP1.4, PS1.AC(N), T1.1, T2.1, T3.1
- new net IIN+: R20.1, SV1.16
- new net N$11: R9.2, T3.2
- new net N$13: R12.2, R9.1
- new net N$14: R12.1, R15.2
- new net N$15: R8.2, T2.2
- new net N$16: R11.2, R8.1
- new net N$18: R14.1, R16.2
- new net N$19: R7.2, T1.2
- new net N$20: R13.1, R18.2
- new net N$21: F4.1, R17.1
- new net N$3: R10.2, R7.1
- new net N$4: R10.1, R13.2
- new net N$5: F4.2, JP1.3
- new net N$6: R11.1, R14.2
- new net VIN-1: IC2A.X3, IC2A.Y0, R1.2, T1.4
- new net VIN-2: IC2A.Y1, IC2A.Y3, R2.2, T2.4
- new net VIN-3: IC2A.Y2, R3.2, T3.4
- net +3V3: now also C2.2, C3.+, IC1A.G1, IC3.VD+, R21.1, X1.3V3; no longer C2.+, C5.2, IC2A.G1, IC3.V+, R14.1, R16.1, U$5.VD+, X2.3V3
- net +5V: now also PS1.+5V; no longer U$4.+5V
- net 5V: now also C4.2, C5.+, C6.2, IC3.VA+, R4.1, X1.5V0; no longer C11.2, C7.+, C8.2, R5.1, U$5.VA+, X2.5V0
- net BS-0: now also IC1A.Y0; no longer IC2A.Y0
- net BS-1: now also IC1A.Y1; no longer IC2A.Y1
- net BS-2: now also IC1A.Y2; no longer IC2A.Y2
- net BS-3: now also IC1A.Y3; no longer IC2A.Y3
- net BS-4: now also IC1A.Y4; no longer IC2A.Y4
- net BS-5: now also IC1A.Y5; no longer IC2A.Y5
- net BS-6: now also IC1A.Y6; no longer IC2A.Y6
- net BS-7: now also IC1A.Y7; no longer IC2A.Y7
- net BS-A: now also IC1A.A, X1.GPIO23; no longer IC2A.A, X2.GPIO23
- net BS-B: now also IC1A.B, X1.TXD; no longer IC2A.B, X2.TXD
- net BS-C: now also IC1A.C, X1.SCL; no longer IC2A.C, X2.SCL
- net C5: now also C12.1, IC3.IIN+, R20.2; no longer C10.1, R7.2, U$5.IIN+
- net CS: now also IC3.CS, X1.SPI_CE0; no longer U$5.CS, X2.SPI_CE0
- net CS-A: now also X1.GPIO17; no longer X2.GPIO17
- net CS-B: now also X1.GPIO18; no longer X2.GPIO18
- net CS-C: now also X1.GPIO27; no longer X2.GPIO27
- net CS-D: now also X1.GPIO22; no longer X2.GPIO22
- net GND: now also C10.1, C12.2, C14.1, C2.1, C3.-, C4.1, C5.-, C7.1, C8.2, IC1A.G2B, IC2A.X0, IC2A.X1, IC2A.X2, IC2P.GND, IC2P.VEE, IC3.AGND, IC3.DGND, IC3.MODE, JP1.5, LED1.C, PS1.GND, R1.1, R19.1, R2.1, R3.1, SV1.15, T1.3, T2.3, T3.3, X1.GND; no longer C10.2, C12.1, C15.1, C2.-, C3.1, C4.2, C5.1, C7.-, C8.1, C9.1, IC1A.X3, IC1A.Y3, IC1P.GND, IC1P.VEE, IC2A.G2B, IC3.V-, JP1.3, JP2.1, PWR.C, R15.2, U$4.GND, U$5.AGND, U$5.DGND, U$5.MODE, X2.GND
- net INH: now also IC1A.G2A, IC2A.INH, X1.SDA; no longer IC1A.INH, IC2A.G2A, X2.SDA
- net INT: now also IC3.INT, X1.GPIO24; no longer U$5.INT, X2.GPIO24
- net N$1: now also IC3.XOUT; no longer U$5.XOUT
- net N$10: now also R15.1, R17.2; no longer IC3.-IN, IC3.OUT, JP1.1
- net N$12: now also IC3.XIN; no longer U$5.XIN
- net N$17: now also C10.2, IC3.VREFIN, IC3.VREFOUT; no longer C6.2, U$5.VREFIN, U$5.VREFOUT
- net N$2: now also F3.1, R16.1; no longer C15.2, IC3.+IN, R15.1, R16.2
- net N$23: now also IC2A.X, R5.2; no longer IC1A.X, R2.2
- net N$38: now also F3.2, JP1.2; no longer F5.2, JP2.2
- net N$39: now also IC2A.Y, R6.2; no longer IC1A.Y, R1.2
- net N$46: now also C8.1, C9.1, IC3.VIN-, R6.1; no longer C14.1, C4.1, R1.1, U$5.VIN-
- net N$7: now also LED1.A, R4.2; no longer PWR.A, R5.2
- net N$8: now also C11.2, IC3.IIN-, R19.2; no longer C9.2, R6.2, U$5.IIN-
- net N$9: now also F2.2, JP1.1; no longer F4.2, JP2.4
- net R1: now also C7.2, C9.2, IC3.VIN+, R5.1; no longer C14.2, C3.2, R2.1, U$5.VIN+
- net RESET: now also C14.2, IC3.RESET, R21.2, X1.GPIO25; no longer C12.2, R14.2, U$5.RESET, X2.GPIO25
- net SCLK: now also IC3.SCLK, X1.SPI_SCLK; no longer U$5.SCLK, X2.SPI_SCLK
- net SDI: now also IC3.SDI, X1.SPI_MOSI; no longer U$5.SDI, X2.SPI_MOSI
- net SDO: now also IC3.SDO, X1.SPI_MISO; no longer U$5.SDO, X2.SPI_MISO
- net VS-A: now also IC2A.A, X1.GPIO04; no longer IC1A.A, X2.GPIO04
- net VS-B: now also IC2A.B, X1.RXD; no longer IC1A.B, X2.RXD
Other:
- note added: "AC Input from electrical panel provides voltage sense and 5V DC power for RPI and electronics. For US 240V split phase use AC1, AC2, Neutral and Ground. For 240V single phase use AC1, Neutral and Ground. For 3 phase use AC1, AC2, AC3, Neutral and Ground."
- note added: "AC1"
- note added: "AC2"
- note added: "AC3"
- note added: "Ground"
- note added: "V1"
- note added: "V2"
- note added: "V3"
- note removed: "AC Line In"
- note removed: "Bias circuit (optional)"
- note removed: "Current board connector"
- moved on the sheet: C1, C10, C11, C12, C14, C4, C6, C8, C9, D1, F1, F4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
